Commit message: Updating

File: src/abb_robot_arm/abb_irb1200_support/urdf/irb1200_5_90_macro.xacro (robot description, xacro)
@@ -53,5 +53,5 @@
           <mesh filename="package://abb_irb1200_support/meshes/irb1200_5_90/visual/link_1.dae"/>
         </geometry>
-         <xacro:colour_orange />
+        <xacro:colour_orange />
       </visual>
     </link>
@@ -72,5 +72,5 @@
           <mesh filename="package://abb_irb1200_support/meshes/irb1200_5_90/visual/link_2.dae"/>
         </geometry>
-         <xacro:colour_orange />
+        <xacro:colour_orange />
       </visual>
     </link>
@@ -91,5 +91,5 @@
           <mesh filename="package://abb_irb1200_support/meshes/irb1200_5_90/visual/link_3.dae"/>
         </geometry>
-         <xacro:colour_orange />
+        <xacro:colour_orange />
       </visual>
     </link>
@@ -110,5 +110,5 @@
           <mesh filename="package://abb_irb1200_support/meshes/irb1200_5_90/visual/link_4.dae"/>
         </geometry>
-         <xacro:colour_orange />
+        <xacro:colour_orange />
       </visual>
     </link>
@@ -129,5 +129,5 @@
           <mesh filename="package://abb_irb1200_support/meshes/irb1200_5_90/visual/link_5.dae"/>
         </geometry>
-         <xacro:colour_orange />
+        <xacro:colour_orange />
       </visual>
     </link>
@@ -148,7 +148,102 @@
           <mesh filename="package://abb_irb1200_support/meshes/irb1200_5_90/visual/link_6.dae"/>
         </geometry>
-         <xacro:colour_orange />
-      </visual>
-    </link>
+        <xacro:colour_orange />
+      </visual>
+    </link>
+    <!-- <link name="${prefix}flange_1">
+      See note 1 in package.xml about the inertial and mass values
+      <inertial>
+        <mass value="0.137"/>
+        <origin xyz="-0.00706 -0.00017 -1.32E-06" rpy="0 0 0"/>
+        <inertia ixx="0.001" ixy="0" ixz="0" iyy="0.001" iyz="0" izz="0.001"/>
+      </inertial>
+      <collision name="collision">
+        <geometry>
+          <mesh filename="package://pick_and_place_env/meshes/flange_1.stl" scale = "0.001 0.001 0.001"/>
+        </geometry>
+      </collision>
+      <visual name="visual">
+        <geometry>
+          <mesh filename="package://pick_and_place_env/meshes/flange_1.stl" scale = "0.001 0.001 0.001"/>
+        </geometry>
+        <xacro:colour_orange />
+      </visual>
+    </link>
+    <link name="${prefix}flange_2">
+      See note 1 in package.xml about the inertial and mass values
+      <inertial>
+        <mass value="0.137"/>
+        <origin xyz="-0.00706 -0.00017 -1.32E-06" rpy="0 0 0"/>
+        <inertia ixx="0.001" ixy="0" ixz="0" iyy="0.001" iyz="0" izz="0.001"/>
+      </inertial>
+      <collision name="collision">
+        <geometry>
+          <mesh filename="package://pick_and_place_env/meshes/flange_2.stl" scale = "0.001 0.001 0.001"/>
+        </geometry>
+      </collision>
+      <visual name="visual">
+        <geometry>
+          <mesh filename="package://pick_and_place_env/meshes/flange_2.stl" scale = "0.001 0.001 0.001"/>
+        </geometry>
+        <xacro:colour_orange />
+      </visual>
+    </link>
+    <link name="${prefix}tool_base">
+      See note 1 in package.xml about the inertial and mass values
+      <inertial>
+        <mass value="0.137"/>
+        <origin xyz="-0.00706 -0.00017 -1.32E-06" rpy="0 0 0"/>
+        <inertia ixx="0.001" ixy="0" ixz="0" iyy="0.001" iyz="0" izz="0.001"/>
+      </inertial>
+      <collision name="collision">
+        <geometry>
+          <mesh filename="package://pick_and_place_env/meshes/tool_base.stl" scale = "0.001 0.001 0.001"/>
+        </geometry>
+      </collision>
+      <visual name="visual">
+        <geometry>
+          <mesh filename="package://pick_and_place_env/meshes/tool_base.stl" scale = "0.001 0.001 0.001"/>
+        </geometry>
+        <xacro:colour_dark_green />
+      </visual>
+    </link>
+    <link name="${prefix}l_finger">
+      See note 1 in package.xml about the inertial and mass values
+      <inertial>
+        <mass value="0.137"/>
+        <origin xyz="-0.00706 -0.00017 -1.32E-06" rpy="0 0 0"/>
+        <inertia ixx="0.001" ixy="0" ixz="0" iyy="0.001" iyz="0" izz="0.001"/>
+      </inertial>
+      <collision name="collision">
+        <geometry>
+          <mesh filename="package://pick_and_place_env/meshes/l_finger.stl" scale = "0.001 0.001 0.001"/>
+        </geometry>
+      </collision>
+      <visual name="visual">
+        <geometry>
+          <mesh filename="package://pick_and_place_env/meshes/l_finger.stl" scale = "0.001 0.001 0.001"/>
+        </geometry>
+        <xacro:colour_gray_60p />
+      </visual>
+    </link>
+    <link name="${prefix}r_finger">
+      See note 1 in package.xml about the inertial and mass values
+      <inertial>
+        <mass value="0.137"/>
+        <origin xyz="3 3 3" rpy="0 0 0"/>
+        <inertia ixx="0.001" ixy="0" ixz="0" iyy="0.001" iyz="0" izz="0.001"/>
+      </inertial>
+      <collision name="collision">
+        <geometry>
+          <mesh filename="package://pick_and_place_env/meshes/r_finger.stl" scale = "0.001 0.001 0.001"/>
+        </geometry>
+      </collision>
+      <visual name="visual">
+        <geometry>
+          <mesh filename="package://pick_and_place_env/meshes/r_finger.stl" scale = "0.001 0.001 0.001"/>
+        </geometry>
+        <xacro:colour_gray_60p />
+      </visual>
+    </link> -->
     <!-- end of link list -->
     <!--  -->
@@ -216,17 +311,45 @@
     </joint>
     <!-- end of joint list -->
-    <!-- ROS-Industrial 'base' frame: base_link to ABB World Coordinates transform -->
     <!-- ROS-Industrial 'flange' frame: attachment point for EEF models -->
-    <link name="${prefix}flange"/>
-    <joint type="fixed" name="${prefix}joint_6-flange">
-      <origin xyz="0 0 0" rpy="0 0 0"/>
+<!--
+    <joint type="fixed" name="${prefix}flange_1">
+      <origin xyz="0 -0.02 0.02" rpy="0 ${pi/2} 0"/>
       <parent link="${prefix}link_6"/>
-      <child link="${prefix}flange"/>
-    </joint>
+      <child link="${prefix}flange_1"/>
+    </joint>
+    <joint type="fixed" name="${prefix}flange_2">
+      <origin xyz="0 0 0" rpy="0 0 0"/>
+      <parent link="${prefix}flange_1"/>
+      <child link="${prefix}flange_2"/>
+    </joint>
+    <joint type="fixed" name="${prefix}tool_base">
+      <origin xyz="0 0 0" rpy="0 0 0"/>
+      <parent link="${prefix}flange_2"/>
+      <child link="${prefix}tool_base"/>
+    </joint>
+    <joint type="revolute" name="${prefix}l_finger">
+      <calibration rising="10"/>
+      <origin xyz="0 0 0" rpy="0 0 0"/>
+      <parent link="${prefix}tool_base"/>
+      <child link="${prefix}l_finger"/>
+      <axis xyz="1 0 0" />
+      <dynamics damping="1.0" friction="1.0"/>
+      <limit effort="1000" lower="0" upper="1" velocity="10.472"/>
+    </joint>
+    <joint type="revolute" name="${prefix}r_finger">
+      <calibration rising="10"/>
+      <origin xyz="0 0 0" rpy="0 0 0"/>
+      <parent link="${prefix}tool_base"/>
+      <child link="${prefix}r_finger"/>
+      <axis xyz="1 0 0" />
+      <dynamics damping="1.0" friction="1.0"/>
+      <limit effort="1000" lower="0" upper="1" velocity="10.472"/>
+    </joint>
+ -->
     <!-- ROS-Industrial 'tool0' frame: all-zeros tool frame -->
     <link name="${prefix}tool0" />
     <joint name="${prefix}link_6-tool0" type="fixed">
       <origin xyz="0 0 0" rpy="0 ${radians(90)} 0" />
-      <parent link="${prefix}flange" />
+      <parent link="${prefix}link_6" />
       <child link="${prefix}tool0" />
     </joint>

File: src/pick_and_place_env/urdf/colours/colour_names.xacro (robot description, xacro)
@@ -22,3 +22,4 @@
   <xacro:property name="c_gray_80p"     value="0.8 0.8 0.8 1" />
   <xacro:property name="c_gray_90p"     value="0.9 0.9 0.9 1" />
+  <xacro:property name="c_dark_green"     value="0 0.5 0 1" />
 </robot>

File: src/pick_and_place_env/urdf/colours/colours.xacro (robot description, xacro)
@@ -15,4 +15,9 @@
     <material name="">
       <color rgba="${c_green}"/>
+    </material>
+  </xacro:macro>
+  <xacro:macro name="colour_dark_green">
+    <material name="">
+      <color rgba="${c_dark_green}"/>
     </material>
   </xacro:macro>

File: src/pick_and_place_env/urdf/conveyor_belt_macro.xacro (robot description, xacro)
@@ -4,4 +4,19 @@
   <xacro:macro name = "Conveyor_belt">
     <!-- link list -->
+    <link name="conveyor_base">
+      <visual>
+        <origin xyz="0 0 0" rpy="0 0 0" />
+        <geometry>
+          <mesh filename="package://pick_and_place_env/meshes/conveyor_base.stl" scale = "0.001 0.001 0.001"/>
+        </geometry>
+        <xacro:colour_gray_30p/>
+      </visual>
+      <collision>
+        <origin xyz="0 0 0" rpy="0 0 0" />
+        <geometry>
+          <mesh filename="package://pick_and_place_env/meshes/conveyor_base.stl" scale = "0.001 0.001 0.001"/>
+        </geometry>
+      </collision>
+    </link>
     <link name="conveyor_belt">
       <visual>
@@ -10,5 +25,5 @@
           <mesh filename="package://pick_and_place_env/meshes/conveyor_belt.stl" scale = "0.001 0.001 0.001"/>
         </geometry>
-        <xacro:colour_gray_50p/>
+        <xacro:colour_gray_90p/>
       </visual>
       <collision>
@@ -23,8 +38,14 @@
     <!--  -->
     <!-- joint list -->
-    <joint name="base_to_conveyor_belt_joint" type="fixed">
-      <origin xyz="0.7 1 0.75" rpy="${pi/2} 0 ${pi/2}"/>
+    <joint name="base_to_conveyor_base_joint" type="fixed">
+      <origin xyz="0.77 1.295 0" rpy="0 0 ${-pi/2}"/>
       <axis xyz="0 0 1"/>
       <parent link="base"/>
+      <child link="conveyor_base"/>
+    </joint>
+    <joint name="conveyor_base_to_conveyor_belt_joint" type="fixed">
+      <origin xyz="0 0 0" rpy="0 0 0"/>
+      <axis xyz="0 0 1"/>
+      <parent link="conveyor_base"/>
       <child link="conveyor_belt"/>
     </joint>

Commit message: Updating

File: src/abb_robot_arm/abb_irb1200_support/urdf/irb1200_5_90_macro.xacro (robot description, xacro)
@@ -312,6 +312,5 @@
     <!-- end of joint list -->
     <!-- ROS-Industrial 'flange' frame: attachment point for EEF models -->
-<!--
-    <joint type="fixed" name="${prefix}flange_1">
+    <!-- <joint type="fixed" name="${prefix}flange_1">
       <origin xyz="0 -0.02 0.02" rpy="0 ${pi/2} 0"/>
       <parent link="${prefix}link_6"/>

Commit message: Updating

File: src/abb_robot_arm/abb_irb1200_support/urdf/irb1200_5_90_macro.xacro (robot description, xacro)
@@ -151,19 +151,20 @@
       </visual>
     </link>
-    <!-- <link name="${prefix}flange_1">
-      See note 1 in package.xml about the inertial and mass values
-      <inertial>
-        <mass value="0.137"/>
-        <origin xyz="-0.00706 -0.00017 -1.32E-06" rpy="0 0 0"/>
-        <inertia ixx="0.001" ixy="0" ixz="0" iyy="0.001" iyz="0" izz="0.001"/>
-      </inertial>
-      <collision name="collision">
-        <geometry>
-          <mesh filename="package://pick_and_place_env/meshes/flange_1.stl" scale = "0.001 0.001 0.001"/>
-        </geometry>
-      </collision>
-      <visual name="visual">
-        <geometry>
-          <mesh filename="package://pick_and_place_env/meshes/flange_1.stl" scale = "0.001 0.001 0.001"/>
+<!--
+    <link name="${prefix}flange_1">
+      See note 1 in package.xml about the inertial and mass values
+      <inertial>
+        <mass value="0.137"/>
+        <origin xyz="-0.00706 -0.00017 -1.32E-06" rpy="0 0 0"/>
+        <inertia ixx="0.001" ixy="0" ixz="0" iyy="0.001" iyz="0" izz="0.001"/>
+      </inertial>
+      <collision name="collision">
+        <geometry>
+          <mesh filename="package://pick_and_place_env/meshes/Common_Flange.stl" scale = "0.001 0.001 0.001"/>
+        </geometry>
+      </collision>
+      <visual name="visual">
+        <geometry>
+          <mesh filename="package://pick_and_place_env/meshes/Common_Flange.stl" scale = "0.001 0.001 0.001"/>
         </geometry>
         <xacro:colour_orange />
@@ -179,12 +180,12 @@
       <collision name="collision">
         <geometry>
-          <mesh filename="package://pick_and_place_env/meshes/flange_2.stl" scale = "0.001 0.001 0.001"/>
-        </geometry>
-      </collision>
-      <visual name="visual">
-        <geometry>
-          <mesh filename="package://pick_and_place_env/meshes/flange_2.stl" scale = "0.001 0.001 0.001"/>
-        </geometry>
-        <xacro:colour_orange />
+          <mesh filename="package://pick_and_place_env/meshes/PB-0013_Flange.stl" scale = "0.001 0.001 0.001"/>
+        </geometry>
+      </collision>
+      <visual name="visual">
+        <geometry>
+          <mesh filename="package://pick_and_place_env/meshes/PB-0013_Flange.stl" scale = "0.001 0.001 0.001"/>
+        </geometry>
+        <xacro:colour_white />
       </visual>
     </link>
@@ -198,12 +199,12 @@
       <collision name="collision">
         <geometry>
-          <mesh filename="package://pick_and_place_env/meshes/tool_base.stl" scale = "0.001 0.001 0.001"/>
-        </geometry>
-      </collision>
-      <visual name="visual">
-        <geometry>
-          <mesh filename="package://pick_and_place_env/meshes/tool_base.stl" scale = "0.001 0.001 0.001"/>
-        </geometry>
-        <xacro:colour_dark_green />
+          <mesh filename="package://pick_and_place_env/meshes/PB-0013_Base.stl" scale = "0.001 0.001 0.001"/>
+        </geometry>
+      </collision>
+      <visual name="visual">
+        <geometry>
+          <mesh filename="package://pick_and_place_env/meshes/PB-0013_Base.stl" scale = "0.001 0.001 0.001"/>
+        </geometry>
+        <xacro:colour_gray_20p />
       </visual>
     </link>
@@ -217,12 +218,12 @@
       <collision name="collision">
         <geometry>
-          <mesh filename="package://pick_and_place_env/meshes/l_finger.stl" scale = "0.001 0.001 0.001"/>
-        </geometry>
-      </collision>
-      <visual name="visual">
-        <geometry>
-          <mesh filename="package://pick_and_place_env/meshes/l_finger.stl" scale = "0.001 0.001 0.001"/>
-        </geometry>
-        <xacro:colour_gray_60p />
+          <mesh filename="package://pick_and_place_env/meshes/PB-0013_Left.stl" scale = "0.001 0.001 0.001"/>
+        </geometry>
+      </collision>
+      <visual name="visual">
+        <geometry>
+          <mesh filename="package://pick_and_place_env/meshes/PB-0013_Left.stl" scale = "0.001 0.001 0.001"/>
+        </geometry>
+        <xacro:colour_gray_40p />
       </visual>
     </link>
@@ -236,12 +237,12 @@
       <collision name="collision">
         <geometry>
-          <mesh filename="package://pick_and_place_env/meshes/r_finger.stl" scale = "0.001 0.001 0.001"/>
-        </geometry>
-      </collision>
-      <visual name="visual">
-        <geometry>
-          <mesh filename="package://pick_and_place_env/meshes/r_finger.stl" scale = "0.001 0.001 0.001"/>
-        </geometry>
-        <xacro:colour_gray_60p />
+          <mesh filename="package://pick_and_place_env/meshes/PB-0013_Right.stl" scale = "0.001 0.001 0.001"/>
+        </geometry>
+      </collision>
+      <visual name="visual">
+        <geometry>
+          <mesh filename="package://pick_and_place_env/meshes/PB-0013_Right.stl" scale = "0.001 0.001 0.001"/>
+        </geometry>
+        <xacro:colour_gray_40p />
       </visual>
     </link> -->
@@ -344,6 +345,5 @@
       <dynamics damping="1.0" friction="1.0"/>
       <limit effort="1000" lower="0" upper="1" velocity="10.472"/>
-    </joint>
- -->
+    </joint> -->
     <!-- ROS-Industrial 'tool0' frame: all-zeros tool frame -->
     <link name="${prefix}tool0" />

File: src/phoxi_camera/urdf/PhoXi3Dscanner_macro.xacro (robot description, xacro)
@@ -10,5 +10,5 @@
           <mesh filename="package://abb_irb1200_support/meshes/irb1200_5_90/visual/camera_stand.stl" scale = "0.001 0.001 0.001"/>
         </geometry>
-        <xacro:colour_gray_50p/>
+        <xacro:colour_gray_70p/>
       </visual>
       <collision>
@@ -25,5 +25,5 @@
           <mesh filename="package://abb_irb1200_support/meshes/irb1200_5_90/visual/camera_support.stl" scale = "0.001 0.001 0.001"/>
         </geometry>
-        <xacro:colour_gray_10p/>
+        <xacro:colour_gray_50p/>
       </visual>
       <collision>

File: src/pick_and_place_env/urdf/conveyor_belt_macro.xacro (robot description, xacro)
@@ -8,5 +8,5 @@
         <origin xyz="0 0 0" rpy="0 0 0" />
         <geometry>
-          <mesh filename="package://pick_and_place_env/meshes/conveyor_base.stl" scale = "0.001 0.001 0.001"/>
+          <mesh filename="package://pick_and_place_env/meshes/Conveyor_Base.stl" scale = "0.001 0.001 0.001"/>
         </geometry>
         <xacro:colour_gray_30p/>
@@ -15,5 +15,5 @@
         <origin xyz="0 0 0" rpy="0 0 0" />
         <geometry>
-          <mesh filename="package://pick_and_place_env/meshes/conveyor_base.stl" scale = "0.001 0.001 0.001"/>
+          <mesh filename="package://pick_and_place_env/meshes/Conveyor_Base.stl" scale = "0.001 0.001 0.001"/>
         </geometry>
       </collision>
@@ -23,12 +23,12 @@
         <origin xyz="0 0 0" rpy="0 0 0" />
         <geometry>
-          <mesh filename="package://pick_and_place_env/meshes/conveyor_belt.stl" scale = "0.001 0.001 0.001"/>
+          <mesh filename="package://pick_and_place_env/meshes/Conveyor_Belt.stl" scale = "0.001 0.001 0.001"/>
         </geometry>
-        <xacro:colour_gray_90p/>
+        <xacro:colour_white/>
       </visual>
       <collision>
         <origin xyz="0 0 0" rpy="0 0 0" />
         <geometry>
-          <mesh filename="package://pick_and_place_env/meshes/conveyor_belt.stl" scale = "0.001 0.001 0.001"/>
+          <mesh filename="package://pick_and_place_env/meshes/Conveyor_Belt.stl" scale = "0.001 0.001 0.001"/>
         </geometry>
       </collision>
