Commit message: Updating

File: src/abb_robot_arm/abb_irb1200_support/urdf/irb1200_5_90_macro.xacro (robot description, xacro)
@@ -4,5 +4,8 @@
   <xacro:include filename="$(find pick_and_place_env)/urdf/colours/colours.xacro"/>
   <xacro:macro name="abb_irb1200_5_90" params="prefix">
-    <!-- link list -->
+    <!--  -->
+    <!--  -->
+    <!--  -->
+    <!-- Robotic arm link list -->
     <link name="${prefix}base">
       <collision name="collision">
@@ -19,5 +22,4 @@
     </link>
     <link name="${prefix}base_link">
-      <!-- See note 1 in package.xml about the inertial and mass values -->
       <inertial>
         <mass value="13.7742"/>
@@ -38,5 +40,4 @@
     </link>
     <link name="${prefix}link_1">
-      <!-- See note 1 in package.xml about the inertial and mass values -->
       <inertial>
         <mass value="11.8419"/>
@@ -57,5 +58,4 @@
     </link>
     <link name="${prefix}link_2">
-      <!-- See note 1 in package.xml about the inertial and mass values -->
       <inertial>
         <mass value="17.5394"/>
@@ -76,5 +76,4 @@
     </link>
     <link name="${prefix}link_3">
-      <!-- See note 1 in package.xml about the inertial and mass values -->
       <inertial>
         <mass value="7.46365"/>
@@ -95,5 +94,4 @@
     </link>
     <link name="${prefix}link_4">
-      <!-- See note 1 in package.xml about the inertial and mass values -->
       <inertial>
         <mass value="2.74436"/>
@@ -114,5 +112,4 @@
     </link>
     <link name="${prefix}link_5">
-      <!-- See note 1 in package.xml about the inertial and mass values -->
       <inertial>
         <mass value="0.62953"/>
@@ -133,5 +130,4 @@
     </link>
     <link name="${prefix}link_6">
-      <!-- See note 1 in package.xml about the inertial and mass values -->
       <inertial>
         <mass value="0.137"/>
@@ -151,7 +147,10 @@
       </visual>
     </link>
-<!--
-    <link name="${prefix}flange_1">
-      See note 1 in package.xml about the inertial and mass values
+    <!-- End of robotic arm link list -->
+    <!--  -->
+    <!--  -->
+    <!--  -->
+    <!-- Gripper link list -->
+    <link name="${prefix}link_flange_1">
       <inertial>
         <mass value="0.137"/>
@@ -171,6 +170,5 @@
       </visual>
     </link>
-    <link name="${prefix}flange_2">
-      See note 1 in package.xml about the inertial and mass values
+    <link name="${prefix}link_flange_2">
       <inertial>
         <mass value="0.137"/>
@@ -190,6 +188,5 @@
       </visual>
     </link>
-    <link name="${prefix}tool_base">
-      See note 1 in package.xml about the inertial and mass values
+    <link name="${prefix}link_tool_base">
       <inertial>
         <mass value="0.137"/>
@@ -209,6 +206,5 @@
       </visual>
     </link>
-    <link name="${prefix}l_finger">
-      See note 1 in package.xml about the inertial and mass values
+    <link name="${prefix}link_l_finger">
       <inertial>
         <mass value="0.137"/>
@@ -228,6 +224,5 @@
       </visual>
     </link>
-    <link name="${prefix}r_finger">
-      See note 1 in package.xml about the inertial and mass values
+    <link name="${prefix}link_r_finger">
       <inertial>
         <mass value="0.137"/>
@@ -246,9 +241,10 @@
         <xacro:colour_gray_40p />
       </visual>
-    </link> -->
-    <!-- end of link list -->
-    <!--  -->
-    <!--  -->
-    <!-- joint list -->
+    </link>
+    <!-- End of gripper link list -->
+    <!--  -->
+    <!--  -->
+    <!--  -->
+    <!-- Robotic arm joint list -->
     <joint type="fixed" name="${prefix}base_link">
       <origin xyz="0.275 0.275 0.726" rpy="0 0 0"/>
@@ -262,5 +258,4 @@
       <parent link="${prefix}base_link"/>
       <child link="${prefix}link_1"/>
-      <!-- See note 2 in package.xml about effort limits and dynamics values -->
       <limit effort="1000" lower="-2.967" upper="2.967" velocity="5.027"/>
       <dynamics damping="50.0" friction="1.0"/>
@@ -271,5 +266,4 @@
       <parent link="${prefix}link_1"/>
       <child link="${prefix}link_2"/>
-      <!-- See note 2 in package.xml about effort limits and dynamics values -->
       <limit effort="1000" lower="-1.745" upper="2.269" velocity="4.189"/>
       <dynamics damping="50.0" friction="1.0"/>
@@ -280,5 +274,4 @@
       <parent link="${prefix}link_2"/>
       <child link="${prefix}link_3"/>
-      <!-- See note 2 in package.xml about effort limits and dynamics values -->
       <limit effort="1000" lower="-3.491" upper="1.222" velocity="5.236"/>
       <dynamics damping="10.0" friction="1.0"/>
@@ -289,5 +282,4 @@
       <parent link="${prefix}link_3"/>
       <child link="${prefix}link_4"/>
-      <!-- See note 2 in package.xml about effort limits and dynamics values -->
       <limit effort="1000" lower="-4.712" upper="4.712" velocity="6.981"/>
       <dynamics damping="5.0" friction="1.0"/>
@@ -298,5 +290,4 @@
       <parent link="${prefix}link_4"/>
       <child link="${prefix}link_5"/>
-      <!-- See note 2 in package.xml about effort limits and dynamics values -->
       <limit effort="1000" lower="-2.269" upper="2.269" velocity="7.069"/>
       <dynamics damping="2.0" friction="1.0"/>
@@ -307,50 +298,46 @@
       <parent link="${prefix}link_5"/>
       <child link="${prefix}link_6"/>
-      <!-- See note 2 in package.xml about effort limits and dynamics values -->
       <limit effort="1000" lower="-6.283" upper="6.283" velocity="10.472"/>
       <dynamics damping="1.0" friction="1.0"/>
     </joint>
-    <!-- end of joint list -->
-    <!-- ROS-Industrial 'flange' frame: attachment point for EEF models -->
-    <!-- <joint type="fixed" name="${prefix}flange_1">
+    <!-- End of robotic arm joint list -->
+    <!--  -->
+    <!--  -->
+    <!--  -->
+    <!-- Gripper joint list -->
+    <joint type="fixed" name="${prefix}joint_flange_1">
       <origin xyz="0 -0.02 0.02" rpy="0 ${pi/2} 0"/>
       <parent link="${prefix}link_6"/>
-      <child link="${prefix}flange_1"/>
-    </joint>
-    <joint type="fixed" name="${prefix}flange_2">
-      <origin xyz="0 0 0" rpy="0 0 0"/>
-      <parent link="${prefix}flange_1"/>
-      <child link="${prefix}flange_2"/>
-    </joint>
-    <joint type="fixed" name="${prefix}tool_base">
-      <origin xyz="0 0 0" rpy="0 0 0"/>
-      <parent link="${prefix}flange_2"/>
-      <child link="${prefix}tool_base"/>
-    </joint>
-    <joint type="revolute" name="${prefix}l_finger">
+      <child link="${prefix}link_flange_1"/>
+    </joint>
+    <joint type="fixed" name="${prefix}joint_flange_2">
+      <origin xyz="0 0 0" rpy="0 0 0"/>
+      <parent link="${prefix}link_flange_1"/>
+      <child link="${prefix}link_flange_2"/>
+    </joint>
+    <joint type="fixed" name="${prefix}joint_tool_base">
+      <origin xyz="0 0 0" rpy="0 0 0"/>
+      <parent link="${prefix}link_flange_2"/>
+      <child link="${prefix}link_tool_base"/>
+    </joint>
+    <joint type="revolute" name="${prefix}joint_l_finger">
       <calibration rising="10"/>
       <origin xyz="0 0 0" rpy="0 0 0"/>
-      <parent link="${prefix}tool_base"/>
-      <child link="${prefix}l_finger"/>
-      <axis xyz="1 0 0" />
+      <parent link="${prefix}link_tool_base"/>
+      <child link="${prefix}link_l_finger"/>
+      <axis xyz="0 1 0" />
       <dynamics damping="1.0" friction="1.0"/>
       <limit effort="1000" lower="0" upper="1" velocity="10.472"/>
     </joint>
-    <joint type="revolute" name="${prefix}r_finger">
+    <joint type="revolute" name="${prefix}joint_r_finger">
       <calibration rising="10"/>
       <origin xyz="0 0 0" rpy="0 0 0"/>
-      <parent link="${prefix}tool_base"/>
-      <child link="${prefix}r_finger"/>
-      <axis xyz="1 0 0" />
+      <parent link="${prefix}link_tool_base"/>
+      <child link="${prefix}link_r_finger"/>
+      <axis xyz="0 -1 0" />
       <dynamics damping="1.0" friction="1.0"/>
       <limit effort="1000" lower="0" upper="1" velocity="10.472"/>
-    </joint> -->
-    <!-- ROS-Industrial 'tool0' frame: all-zeros tool frame -->
-    <link name="${prefix}tool0" />
-    <joint name="${prefix}link_6-tool0" type="fixed">
-      <origin xyz="0 0 0" rpy="0 ${radians(90)} 0" />
-      <parent link="${prefix}link_6" />
-      <child link="${prefix}tool0" />
-    </joint>
+    </joint>
+    <!-- End of gripper joint list -->
   </xacro:macro>
 </robot>
