Commit message: Updating

File: src/abb_robot_arm/abb_irb1200_support/urdf/irb1200_5_90_macro.xacro (robot description, xacro)
@@ -3,23 +3,35 @@
   <xacro:include filename="$(find abb_resources)/urdf/common_materials.xacro"/>
   <xacro:include filename="$(find pick_and_place_env)/urdf/colours/colours.xacro"/>
-  <xacro:macro name="abb_irb1200_5_90" params="prefix">
+  <xacro:macro name="abb_irb1200_5_90">
     <!--  -->
     <!--  -->
     <!--  -->
     <!-- Robotic arm link list -->
-    <link name="${prefix}base">
-      <collision name="collision">
+    <!-- BASE -->
+    <link name="base">
+      <visual name="visual">
         <geometry>
           <mesh filename="package://abb_irb1200_support/meshes/irb1200_5_90/visual/robot_stand.stl" scale = "0.001 0.001 0.001"/>
         </geometry>
-      </collision>
-      <visual name="visual">
+        <xacro:colour_gray_50p/>
+      </visual>
+      <collision name="collision">
         <geometry>
           <mesh filename="package://abb_irb1200_support/meshes/irb1200_5_90/visual/robot_stand.stl" scale = "0.001 0.001 0.001"/>
         </geometry>
-        <xacro:colour_gray_50p/>
-      </visual>
-    </link>
-    <link name="${prefix}base_link">
+      </collision>
+    </link>
+    <!-- BASE_LINK -->
+    <link name="base_link">
+      <visual name="visual">
+        <geometry>
+          <mesh filename="package://abb_irb1200_support/meshes/irb1200_5_90/visual/base_link.dae"/>
+        </geometry>
+      </visual>
+      <collision name="collision">
+        <geometry>
+          <mesh filename="package://abb_irb1200_support/meshes/irb1200_5_90/collision/base_link.stl"/>
+        </geometry>
+      </collision>
       <inertial>
         <mass value="13.7742"/>
@@ -27,17 +39,17 @@
         <inertia ixx="0.101998" ixy="0.000495482" ixz="0.000311158" iyy="0.13969" iyz="-0.000245375" izz="0.130433"/>
       </inertial>
-      <collision name="collision">
-        <geometry>
-          <mesh filename="package://abb_irb1200_support/meshes/irb1200_5_90/collision/base_link.stl"/>
-        </geometry>
-      </collision>
-      <visual name="visual">
-        <xacro:colour_orange />
-        <geometry>
-          <mesh filename="package://abb_irb1200_support/meshes/irb1200_5_90/visual/base_link.dae"/>
-        </geometry>
-      </visual>
-    </link>
-    <link name="${prefix}link_1">
+    </link>
+    <!-- LINK 1 -->
+    <link name="link_1">
+      <visual name="visual">
+        <geometry>
+          <mesh filename="package://abb_irb1200_support/meshes/irb1200_5_90/visual/link_1.dae"/>
+        </geometry>
+      </visual>
+      <collision>
+        <geometry>
+          <mesh filename="package://abb_irb1200_support/meshes/irb1200_5_90/collision/link_1.stl"/>
+        </geometry>
+      </collision>
       <inertial>
         <mass value="11.8419"/>
@@ -45,17 +57,17 @@
         <inertia ixx="0.11194" ixy="-4.54988e-05" ixz="0.000280961" iyy="0.0915159" iyz="-0.000109905" izz="0.0876456"/>
       </inertial>
-      <collision name="collision">
-        <geometry>
-          <mesh filename="package://abb_irb1200_support/meshes/irb1200_5_90/collision/link_1.stl"/>
-        </geometry>
-      </collision>
-      <visual name="visual">
-        <geometry>
-          <mesh filename="package://abb_irb1200_support/meshes/irb1200_5_90/visual/link_1.dae"/>
-        </geometry>
-        <xacro:colour_orange />
-      </visual>
-    </link>
-    <link name="${prefix}link_2">
+    </link>
+    <!-- LINK 2 -->
+    <link name="link_2">
+      <visual name="visual">
+        <geometry>
+          <mesh filename="package://abb_irb1200_support/meshes/irb1200_5_90/visual/link_2.dae"/>
+        </geometry>
+      </visual>
+      <collision name="collision">
+        <geometry>
+          <mesh filename="package://abb_irb1200_support/meshes/irb1200_5_90/collision/link_2.stl"/>
+        </geometry>
+      </collision>
       <inertial>
         <mass value="17.5394"/>
@@ -63,17 +75,18 @@
         <inertia ixx="0.493558" ixy="1.32136e-05" ixz="0.000209024" iyy="0.462939" iyz="-0.00179901" izz="0.0894214"/>
       </inertial>
-      <collision name="collision">
-        <geometry>
-          <mesh filename="package://abb_irb1200_support/meshes/irb1200_5_90/collision/link_2.stl"/>
-        </geometry>
-      </collision>
-      <visual name="visual">
-        <geometry>
-          <mesh filename="package://abb_irb1200_support/meshes/irb1200_5_90/visual/link_2.dae"/>
+    </link>
+    <!-- LINK 3 -->
+    <link name="link_3">
+      <visual name="visual">
+        <geometry>
+          <mesh filename="package://abb_irb1200_support/meshes/irb1200_5_90/visual/link_3.dae"/>
         </geometry>
         <xacro:colour_orange />
       </visual>
-    </link>
-    <link name="${prefix}link_3">
+      <collision name="collision">
+        <geometry>
+          <mesh filename="package://abb_irb1200_support/meshes/irb1200_5_90/collision/link_3.stl"/>
+        </geometry>
+      </collision>
       <inertial>
         <mass value="7.46365"/>
@@ -81,17 +94,17 @@
         <inertia ixx="0.0252424" ixy="0.000142737" ixz="-0.00565542" iyy="0.0906438" iyz="0.000142213" izz="0.0825079"/>
       </inertial>
-      <collision name="collision">
-        <geometry>
-          <mesh filename="package://abb_irb1200_support/meshes/irb1200_5_90/collision/link_3.stl"/>
-        </geometry>
-      </collision>
-      <visual name="visual">
-        <geometry>
-          <mesh filename="package://abb_irb1200_support/meshes/irb1200_5_90/visual/link_3.dae"/>
-        </geometry>
-        <xacro:colour_orange />
-      </visual>
-    </link>
-    <link name="${prefix}link_4">
+    </link>
+    <!-- LINK 4 -->
+    <link name="link_4">
+      <visual name="visual">
+        <geometry>
+          <mesh filename="package://abb_irb1200_support/meshes/irb1200_5_90/visual/link_4.dae"/>
+        </geometry>
+      </visual>
+      <collision name="collision">
+        <geometry>
+          <mesh filename="package://abb_irb1200_support/meshes/irb1200_5_90/collision/link_4.stl"/>
+        </geometry>
+      </collision>
       <inertial>
         <mass value="2.74436"/>
@@ -99,17 +112,17 @@
         <inertia ixx="0.00573099" ixy="-0.000131119" ixz="0.000380232" iyy="0.0118352" iyz="-2.26565e-05" izz="0.0114428"/>
       </inertial>
-      <collision name="collision">
-        <geometry>
-          <mesh filename="package://abb_irb1200_support/meshes/irb1200_5_90/collision/link_4.stl"/>
-        </geometry>
-      </collision>
-      <visual name="visual">
-        <geometry>
-          <mesh filename="package://abb_irb1200_support/meshes/irb1200_5_90/visual/link_4.dae"/>
-        </geometry>
-        <xacro:colour_orange />
-      </visual>
-    </link>
-    <link name="${prefix}link_5">
+    </link>
+    <!-- LINK 5 -->
+    <link name="link_5">
+      <visual name="visual">
+        <geometry>
+          <mesh filename="package://abb_irb1200_support/meshes/irb1200_5_90/visual/link_5.dae"/>
+        </geometry>
+      </visual>
+      <collision name="collision">
+        <geometry>
+          <mesh filename="package://abb_irb1200_support/meshes/irb1200_5_90/collision/link_5.stl"/>
+        </geometry>
+      </collision>
       <inertial>
         <mass value="0.62953"/>
@@ -117,17 +130,17 @@
         <inertia ixx="0.000502815" ixy="-1.03173e-05" ixz="-8.74347e-08" iyy="0.00108856" iyz="2.07657e-07" izz="0.000918873"/>
       </inertial>
-      <collision name="collision">
-        <geometry>
-          <mesh filename="package://abb_irb1200_support/meshes/irb1200_5_90/collision/link_5.stl"/>
-        </geometry>
-      </collision>
-      <visual name="visual">
-        <geometry>
-          <mesh filename="package://abb_irb1200_support/meshes/irb1200_5_90/visual/link_5.dae"/>
-        </geometry>
-        <xacro:colour_orange />
-      </visual>
-    </link>
-    <link name="${prefix}link_6">
+    </link>
+    <!-- LINK 6 -->
+    <link name="link_6">
+      <visual name="visual">
+        <geometry>
+          <mesh filename="package://abb_irb1200_support/meshes/irb1200_5_90/visual/link_6.dae"/>
+        </geometry>
+      </visual>
+      <collision name="collision">
+        <geometry>
+          <mesh filename="package://abb_irb1200_support/meshes/irb1200_5_90/collision/link_6.stl"/>
+        </geometry>
+      </collision>
       <inertial>
         <mass value="0.137"/>
@@ -135,15 +148,4 @@
         <inertia ixx="0.001" ixy="0" ixz="0" iyy="0.001" iyz="0" izz="0.001"/>
       </inertial>
-      <collision name="collision">
-        <geometry>
-          <mesh filename="package://abb_irb1200_support/meshes/irb1200_5_90/collision/link_6.stl"/>
-        </geometry>
-      </collision>
-      <visual name="visual">
-        <geometry>
-          <mesh filename="package://abb_irb1200_support/meshes/irb1200_5_90/visual/link_6.dae"/>
-        </geometry>
-        <xacro:colour_orange />
-      </visual>
     </link>
     <!-- End of robotic arm link list -->
@@ -151,193 +153,70 @@
     <!--  -->
     <!--  -->
-    <!-- Gripper link list -->
-    <link name="${prefix}link_flange_1">
-      <inertial>
-        <mass value="0.137"/>
-        <origin xyz="-0.00706 -0.00017 -1.32E-06" rpy="0 0 0"/>
-        <inertia ixx="0.001" ixy="0" ixz="0" iyy="0.001" iyz="0" izz="0.001"/>
-      </inertial>
-      <collision name="collision">
-        <geometry>
-          <mesh filename="package://pick_and_place_env/meshes/Common_Flange.stl" scale = "0.001 0.001 0.001"/>
-        </geometry>
-      </collision>
-      <visual name="visual">
-        <geometry>
-          <mesh filename="package://pick_and_place_env/meshes/Common_Flange.stl" scale = "0.001 0.001 0.001"/>
-        </geometry>
-        <xacro:colour_orange />
-      </visual>
-    </link>
-    <link name="${prefix}link_flange_2">
-      <inertial>
-        <mass value="0.137"/>
-        <origin xyz="-0.00706 -0.00017 -1.32E-06" rpy="0 0 0"/>
-        <inertia ixx="0.001" ixy="0" ixz="0" iyy="0.001" iyz="0" izz="0.001"/>
-      </inertial>
-      <collision name="collision">
-        <geometry>
-          <mesh filename="package://pick_and_place_env/meshes/PB-0013_Flange.stl" scale = "0.001 0.001 0.001"/>
-        </geometry>
-      </collision>
-      <visual name="visual">
-        <geometry>
-          <mesh filename="package://pick_and_place_env/meshes/PB-0013_Flange.stl" scale = "0.001 0.001 0.001"/>
-        </geometry>
-        <xacro:colour_white />
-      </visual>
-    </link>
-    <link name="${prefix}link_tool_base">
-      <inertial>
-        <mass value="0.137"/>
-        <origin xyz="-0.00706 -0.00017 -1.32E-06" rpy="0 0 0"/>
-        <inertia ixx="0.001" ixy="0" ixz="0" iyy="0.001" iyz="0" izz="0.001"/>
-      </inertial>
-      <collision name="collision">
-        <geometry>
-          <mesh filename="package://pick_and_place_env/meshes/PB-0013_Base.stl" scale = "0.001 0.001 0.001"/>
-        </geometry>
-      </collision>
-      <visual name="visual">
-        <geometry>
-          <mesh filename="package://pick_and_place_env/meshes/PB-0013_Base.stl" scale = "0.001 0.001 0.001"/>
-        </geometry>
-        <xacro:colour_gray_20p />
-      </visual>
-    </link>
-    <link name="${prefix}link_l_finger">
-      <inertial>
-        <mass value="0.137"/>
-        <origin xyz="-0.00706 -0.00017 -1.32E-06" rpy="0 0 0"/>
-        <inertia ixx="0.001" ixy="0" ixz="0" iyy="0.001" iyz="0" izz="0.001"/>
-      </inertial>
-      <collision name="collision">
-        <geometry>
-          <mesh filename="package://pick_and_place_env/meshes/PB-0013_Left.stl" scale = "0.001 0.001 0.001"/>
-        </geometry>
-      </collision>
-      <visual name="visual">
-        <geometry>
-          <mesh filename="package://pick_and_place_env/meshes/PB-0013_Left.stl" scale = "0.001 0.001 0.001"/>
-        </geometry>
-        <xacro:colour_gray_40p />
-      </visual>
-    </link>
-    <link name="${prefix}link_r_finger">
-      <inertial>
-        <mass value="0.137"/>
-        <origin xyz="3 3 3" rpy="0 0 0"/>
-        <inertia ixx="0.001" ixy="0" ixz="0" iyy="0.001" iyz="0" izz="0.001"/>
-      </inertial>
-      <collision name="collision">
-        <geometry>
-          <mesh filename="package://pick_and_place_env/meshes/PB-0013_Right.stl" scale = "0.001 0.001 0.001"/>
-        </geometry>
-      </collision>
-      <visual name="visual">
-        <geometry>
-          <mesh filename="package://pick_and_place_env/meshes/PB-0013_Right.stl" scale = "0.001 0.001 0.001"/>
-        </geometry>
-        <xacro:colour_gray_40p />
-      </visual>
-    </link>
-    <!-- End of gripper link list -->
-    <!--  -->
-    <!--  -->
-    <!--  -->
     <!-- Robotic arm joint list -->
-    <joint type="fixed" name="${prefix}base_link">
+    <!--  -->
+    <!--  -->
+    <!--  -->
+    <!-- JOINT BASE_LINK -->
+    <joint type="fixed" name="base_link">
       <origin xyz="0.275 0.275 0.726" rpy="0 0 0"/>
       <axis xyz="0 0 0"/>
-      <parent link="${prefix}base"/>
-      <child link="${prefix}base_link"/>
-    </joint>
-    <joint type="revolute" name="${prefix}joint_1">
+      <parent link="base"/>
+      <child link="base_link"/>
+    </joint>
+    <!-- JOINT 1 -->
+    <joint type="revolute" name="joint_1">
       <origin xyz="0 0 0.3991" rpy="0 0 0"/>
       <axis xyz="0 0 1"/>
-      <parent link="${prefix}base_link"/>
-      <child link="${prefix}link_1"/>
+      <parent link="base_link"/>
+      <child link="link_1"/>
       <limit effort="1000" lower="-2.967" upper="2.967" velocity="5.027"/>
       <dynamics damping="50.0" friction="1.0"/>
     </joint>
-    <joint type="revolute" name="${prefix}joint_2">
+    <!-- JOINT 2 -->
+    <joint type="revolute" name="joint_2">
       <origin xyz="0 0 0" rpy="0 0 0"/>
       <axis xyz="0 1 0"/>
-      <parent link="${prefix}link_1"/>
-      <child link="${prefix}link_2"/>
+      <parent link="link_1"/>
+      <child link="link_2"/>
       <limit effort="1000" lower="-1.745" upper="2.269" velocity="4.189"/>
       <dynamics damping="50.0" friction="1.0"/>
     </joint>
-    <joint type="revolute" name="${prefix}joint_3">
+    <!-- JOINT 3 -->
+    <joint type="revolute" name="joint_3">
       <origin xyz="0 0 0.448" rpy="0 0 0"/>
       <axis xyz="0 1 0"/>
-      <parent link="${prefix}link_2"/>
-      <child link="${prefix}link_3"/>
+      <parent link="link_2"/>
+      <child link="link_3"/>
       <limit effort="1000" lower="-3.491" upper="1.222" velocity="5.236"/>
       <dynamics damping="10.0" friction="1.0"/>
     </joint>
-    <joint type="revolute" name="${prefix}joint_4">
+    <!-- JOINT 4 -->
+    <joint type="revolute" name="joint_4">
       <origin xyz="0 0 0.042" rpy="0 0 0"/>
       <axis xyz="1 0 0"/>
-      <parent link="${prefix}link_3"/>
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
File: src/phoxi_camera/urdf/PhoXi3Dscanner_macro.xacro (robot description, xacro)
@@ -2,16 +2,14 @@
 <robot xmlns:xacro="http://ros.org/wiki/xacro">
   <xacro:include filename="$(find pick_and_place_env)/urdf/colours/colours.xacro"/>
-  <xacro:macro name = "PhoXi3Dscanner" params ="scanner_parent scanner_name *scanner_origin sensor_parent sensor_name *sensor_origin *visual *collision">
+  <xacro:macro name = "PhoXi3Dscanner">
     <!-- link list -->
     <link name="camera_stand">
       <visual>
-        <origin xyz="0 0 0" rpy="0 0 0" />
         <geometry>
           <mesh filename="package://abb_irb1200_support/meshes/irb1200_5_90/visual/camera_stand.stl" scale = "0.001 0.001 0.001"/>
         </geometry>
-        <xacro:colour_gray_70p/>
+        <!-- <xacro:colour_gray_70p/> -->
       </visual>
       <collision>
-        <origin xyz="0 0 0" rpy="0 0 0" />
         <geometry>
           <mesh filename="package://abb_irb1200_support/meshes/irb1200_5_90/visual/camera_stand.stl" scale = "0.001 0.001 0.001"/>
@@ -21,12 +19,10 @@
     <link name="camera_support">
       <visual>
-        <origin xyz="0 0 0" rpy="0 0 0" />
         <geometry>
           <mesh filename="package://abb_irb1200_support/meshes/irb1200_5_90/visual/camera_support.stl" scale = "0.001 0.001 0.001"/>
         </geometry>
-        <xacro:colour_gray_50p/>
+        <!-- <xacro:colour_gray_50p/> -->
       </visual>
       <collision>
-        <origin xyz="0 0 0" rpy="0 0 0" />
         <geometry>
           <mesh filename="package://abb_irb1200_support/meshes/irb1200_5_90/visual/camera_support.stl" scale = "0.001 0.001 0.001"/>
@@ -34,9 +30,9 @@
       </collision>
     </link>
-    <link name="${scanner_name}">
+    <link name="PhoXi3Dscanner">
       <visual>
         <origin xyz="0 0 0" rpy="0 1.5707 0" />
         <geometry>
-          <xacro:insert_block name="visual" />
+          <mesh filename="package://phoxi_camera/meshes/visual/PhoXi_S.f.STL" scale = "0.001 0.001 0.001"/>
         </geometry>
         <xacro:colour_gray_30p/>
@@ -45,9 +41,9 @@
         <origin xyz="0 0 0" rpy="0 1.5707 0" />
         <geometry>
-          <xacro:insert_block name="collision" />
+          <mesh filename="package://phoxi_camera/meshes/collision/PhoXi_L.c.STL" scale = "0.001 0.001 0.001"/>
         </geometry>
       </collision>
     </link>
-    <link name="${sensor_name}"/>
+    <link name="PhoXi3Dscanner_sensor"/>
     <!-- end of link list -->
     <!--  -->
@@ -66,14 +62,14 @@
       <child link="camera_support"/>
     </joint>
-    <joint name="camera_support_to_${scanner_name}_joint" type="fixed">
+    <joint name="camera_support_to_PhoXi3Dscanner_joint" type="fixed">
       <origin xyz="0 0.04 0.02" rpy="${pi} 0 ${-pi/2}"/>
       <axis xyz="0 0 1"/>
       <parent link="camera_support"/>
-      <child link="${scanner_name}"/>
+      <child link="PhoXi3Dscanner"/>
     </joint>
-    <joint name="${sensor_parent}_to_${sensor_name}_joint" type="fixed">
-      <parent link="${sensor_parent}"/>
-      <child link="${sensor_name}"/>
-      <xacro:insert_block name="sensor_origin" />
+    <joint name="PhoXi3Dscanner_to_PhoXi3Dscanner_sensor_joint" type="fixed">
+      <origin xyz="-0.1173845315 0.0299 0.005287752939" rpy="0 ${-15.45/180*pi} ${pi}" />
+      <parent link="PhoXi3Dscanner"/>
+      <child link="PhoXi3Dscanner_sensor"/>
     </joint>
     <!-- end of joint list -->

File: src/pick_and_place_env/urdf/conveyor_belt_macro.xacro (robot description, xacro)
@@ -6,12 +6,10 @@
     <link name="conveyor_base">
       <visual>
-        <origin xyz="0 0 0" rpy="0 0 0" />
         <geometry>
           <mesh filename="package://pick_and_place_env/meshes/Conveyor_Base.stl" scale = "0.001 0.001 0.001"/>
         </geometry>
-        <xacro:colour_gray_30p/>
+        <!-- <xacro:colour_gray_30p/> -->
       </visual>
-      <collision>
-        <origin xyz="0 0 0" rpy="0 0 0" />
+      <collision name="collision">
         <geometry>
           <mesh filename="package://pick_and_place_env/meshes/Conveyor_Base.stl" scale = "0.001 0.001 0.001"/>
@@ -21,12 +19,10 @@
     <link name="conveyor_belt">
       <visual>
-        <origin xyz="0 0 0" rpy="0 0 0" />
         <geometry>
           <mesh filename="package://pick_and_place_env/meshes/Conveyor_Belt.stl" scale = "0.001 0.001 0.001"/>
         </geometry>
-        <xacro:colour_white/>
+        <!-- <xacro:colour_white/> -->
       </visual>
       <collision>
-        <origin xyz="0 0 0" rpy="0 0 0" />
         <geometry>
           <mesh filename="package://pick_and_place_env/meshes/Conveyor_Belt.stl" scale = "0.001 0.001 0.001"/>

File: src/pick_and_place_env/urdf/environment.xacro (robot description, xacro)
@@ -1,13 +1,10 @@
-<?xml version="1.0" ?>
+<?xml version="1.0"?>
 <robot name="abb_irb1200_5_90" xmlns:xacro="http://ros.org/wiki/xacro">
   <xacro:include filename="$(find abb_irb1200_support)/urdf/irb1200_5_90_macro.xacro"/>
-  <xacro:abb_irb1200_5_90 prefix=""/>
-  <xacro:include filename="$(find phoxi_camera)/urdf/PhoXi3Dscanner_values.xacro"/>  <!--Scanner values-->
-  <xacro:include filename="$(find phoxi_camera)/urdf/PhoXi3Dscanner_macro.xacro"/>  <!--Scanner macro-->
-  <xacro:PhoXi3Dscanner scanner_parent = "base_link" scanner_name = "PhoXi3Dscanner" sensor_parent = "PhoXi3Dscanner" sensor_name = "PhoXi3Dscanner_sensor" >
-    <origin xyz="0 0 0" rpy="0 0 0" />    <!--PhoXi3Dscanner origin-->
-    <xacro:PhoXi3DscannerS_default_sensor_origin />    <!--Extrinsic calibration data-->
-    <xacro:PhoXi3DscannerS_meshes />    <!--meshes-->
-  </xacro:PhoXi3Dscanner>
+  <xacro:abb_irb1200_5_90 />
+  <xacro:include filename="$(find pick_and_place_env)/urdf/two_finger_gripper_macro.xacro"/>
+  <xacro:two_finger_gripper />
+  <xacro:include filename="$(find phoxi_camera)/urdf/PhoXi3Dscanner_macro.xacro"/>
+  <xacro:PhoXi3Dscanner />
   <xacro:include filename="$(find pick_and_place_env)/urdf/conveyor_belt_macro.xacro"/>
   <xacro:Conveyor_belt/>
