Commit message: Creating the entire pilot line env

File: src/abb_robot_arm/abb_irb1200_support/urdf/irb1200_5_90_macro.xacro (robot description, xacro)
@@ -8,18 +8,4 @@
     <!--  -->
     <!-- Robotic arm link list -->
-    <!-- BASE -->
-    <link name="base">
-      <visual name="visual">
-        <geometry>
-          <mesh filename="package://abb_irb1200_support/meshes/irb1200_5_90/visual/robot_stand.stl" scale = "0.001 0.001 0.001"/>
-        </geometry>
-        <xacro:colour_gray_50p/>
-      </visual>
-      <collision name="collision">
-        <geometry>
-          <mesh filename="package://abb_irb1200_support/meshes/irb1200_5_90/visual/robot_stand.stl" scale = "0.001 0.001 0.001"/>
-        </geometry>
-      </collision>
-    </link>
     <!-- BASE_LINK -->
     <link name="base_link">
@@ -159,7 +145,7 @@
     <!-- JOINT BASE_LINK -->
     <joint type="fixed" name="base_link">
-      <origin xyz="0.275 0.275 0.726" rpy="0 0 0"/>
+      <origin xyz="0 0 0.726" rpy="0 0 0"/>
       <axis xyz="0 0 0"/>
-      <parent link="base"/>
+      <parent link="Fixed_frame"/>
       <child link="base_link"/>
     </joint>

File: src/phoxi_camera/urdf/PhoXi3Dscanner_macro.xacro (robot description, xacro)
@@ -4,30 +4,4 @@
   <xacro:macro name = "PhoXi3Dscanner">
     <!-- link list -->
-    <link name="camera_stand">
-      <visual>
-        <geometry>
-          <mesh filename="package://abb_irb1200_support/meshes/irb1200_5_90/visual/camera_stand.stl" scale = "0.001 0.001 0.001"/>
-        </geometry>
-        <!-- <xacro:colour_gray_70p/> -->
-      </visual>
-      <collision>
-        <geometry>
-          <mesh filename="package://abb_irb1200_support/meshes/irb1200_5_90/visual/camera_stand.stl" scale = "0.001 0.001 0.001"/>
-        </geometry>
-      </collision>
-    </link>
-    <link name="camera_support">
-      <visual>
-        <geometry>
-          <mesh filename="package://abb_irb1200_support/meshes/irb1200_5_90/visual/camera_support.stl" scale = "0.001 0.001 0.001"/>
-        </geometry>
-        <!-- <xacro:colour_gray_50p/> -->
-      </visual>
-      <collision>
-        <geometry>
-          <mesh filename="package://abb_irb1200_support/meshes/irb1200_5_90/visual/camera_support.stl" scale = "0.001 0.001 0.001"/>
-        </geometry>
-      </collision>
-    </link>
     <link name="PhoXi3Dscanner">
       <visual>
@@ -41,5 +15,5 @@
         <origin xyz="0 0 0" rpy="0 1.5707 0" />
         <geometry>
-          <mesh filename="package://phoxi_camera/meshes/collision/PhoXi_L.c.STL" scale = "0.001 0.001 0.001"/>
+          <mesh filename="package://phoxi_camera/meshes/collision/PhoXi_S.c.STL" scale = "0.001 0.001 0.001"/>
         </geometry>
       </collision>
@@ -50,20 +24,7 @@
     <!--  -->
     <!-- joint list -->
-    <joint name="base_to_camera_stand_joint" type="fixed">
-      <origin xyz="1.535 1.02 0" rpy="0 0 ${pi}"/>
-      <axis xyz="0 0 1"/>
-      <parent link="base"/>
-      <child link="camera_stand"/>
-    </joint>
-    <joint name="camera_stand_to_camera_support_joint" type="fixed">
-      <origin xyz="0.515 0.145 1.202" rpy="0 0 ${pi}"/>
-      <axis xyz="0 0 1"/>
-      <parent link="camera_stand"/>
-      <child link="camera_support"/>
-    </joint>
     <joint name="camera_support_to_PhoXi3Dscanner_joint" type="fixed">
-      <origin xyz="0 0.04 0.02" rpy="${pi} 0 ${-pi/2}"/>
-      <axis xyz="0 0 1"/>
-      <parent link="camera_support"/>
+      <origin xyz="0.745 0.640 1.231" rpy="${pi} 0 ${-pi/2}"/>
+      <parent link="Fixed_frame"/>
       <child link="PhoXi3Dscanner"/>
     </joint>

File: src/pick_and_place_env/urdf/conveyor_belt_macro.xacro (robot description, xacro)
@@ -7,5 +7,5 @@
       <visual>
         <geometry>
-          <mesh filename="package://pick_and_place_env/meshes/Conveyor_Base.stl" scale = "0.001 0.001 0.001"/>
+          <mesh filename="package://pick_and_place_env/meshes/Conveyor_Base.dae" scale = "0.001 0.001 0.001"/>
         </geometry>
         <!-- <xacro:colour_gray_30p/> -->
@@ -13,5 +13,5 @@
       <collision name="collision">
         <geometry>
-          <mesh filename="package://pick_and_place_env/meshes/Conveyor_Base.stl" scale = "0.001 0.001 0.001"/>
+          <mesh filename="package://pick_and_place_env/meshes/Conveyor_Base.dae" scale = "0.001 0.001 0.001"/>
         </geometry>
       </collision>
@@ -20,5 +20,5 @@
       <visual>
         <geometry>
-          <mesh filename="package://pick_and_place_env/meshes/Conveyor_Belt.stl" scale = "0.001 0.001 0.001"/>
+          <mesh filename="package://pick_and_place_env/meshes/Conveyor_Belt.dae" scale = "0.001 0.001 0.001"/>
         </geometry>
         <!-- <xacro:colour_white/> -->
@@ -26,5 +26,5 @@
       <collision>
         <geometry>
-          <mesh filename="package://pick_and_place_env/meshes/Conveyor_Belt.stl" scale = "0.001 0.001 0.001"/>
+          <mesh filename="package://pick_and_place_env/meshes/Conveyor_Belt.dae" scale = "0.001 0.001 0.001"/>
         </geometry>
       </collision>
@@ -35,5 +35,5 @@
     <!-- joint list -->
     <joint name="base_to_conveyor_base_joint" type="fixed">
-      <origin xyz="0.77 1.295 0" rpy="0 0 ${-pi/2}"/>
+      <origin xyz="0.495 1.020 0" rpy="0 0 ${-pi/2}"/>
       <axis xyz="0 0 1"/>
       <parent link="base"/>

File: src/pick_and_place_env/urdf/environment.xacro (robot description, xacro)
@@ -1,4 +1,6 @@
 <?xml version="1.0"?>
 <robot name="abb_irb1200_5_90" xmlns:xacro="http://ros.org/wiki/xacro">
+  <xacro:include filename="$(find pick_and_place_env)/urdf/Fixed_parts_macro.xacro"/>
+  <xacro:Fixed_parts/>
   <xacro:include filename="$(find abb_irb1200_support)/urdf/irb1200_5_90_macro.xacro"/>
   <xacro:abb_irb1200_5_90 />
@@ -7,5 +9,3 @@
   <xacro:include filename="$(find phoxi_camera)/urdf/PhoXi3Dscanner_macro.xacro"/>
   <xacro:PhoXi3Dscanner />
-  <xacro:include filename="$(find pick_and_place_env)/urdf/conveyor_belt_macro.xacro"/>
-  <xacro:Conveyor_belt/>
 </robot>

File: src/pick_and_place_env/urdf/two_finger_gripper_macro.xacro (robot description, xacro)
@@ -13,5 +13,5 @@
           <mesh filename="package://pick_and_place_env/meshes/Common_Flange.stl" scale = "0.001 0.001 0.001"/>
         </geometry>
-        <!-- <xacro:colour_orange /> -->
+        <xacro:colour_orange />
       </visual>
       <collision name="collision">
@@ -30,5 +30,5 @@
           <mesh filename="package://pick_and_place_env/meshes/PB-0013_Flange.stl" scale = "0.001 0.001 0.001"/>
         </geometry>
-        <!-- <xacro:colour_white /> -->
+        <xacro:colour_white />
       </visual>
       <collision name="collision">
@@ -47,5 +47,5 @@
           <mesh filename="package://pick_and_place_env/meshes/PB-0013_Base.stl" scale = "0.001 0.001 0.001"/>
         </geometry>
-        <!-- <xacro:colour_gray_20p /> -->
+        <xacro:colour_gray_20p />
       </visual>
       <collision name="collision">
@@ -64,5 +64,5 @@
           <mesh filename="package://pick_and_place_env/meshes/PB-0013_Left.stl" scale = "0.001 0.001 0.001"/>
         </geometry>
-        <!-- <xacro:colour_gray_40p /> -->
+        <xacro:colour_gray_40p />
       </visual>
       <collision name="collision">
@@ -81,5 +81,5 @@
           <mesh filename="package://pick_and_place_env/meshes/PB-0013_Right.stl" scale = "0.001 0.001 0.001"/>
         </geometry>
-        <!-- <xacro:colour_gray_40p /> -->
+        <xacro:colour_gray_40p />
       </visual>
       <collision name="collision">

Commit message: Add large file

File: src/abb_robot_arm/abb_irb1200_support/urdf/irb1200_5_90_macro.xacro (robot description, xacro)
@@ -1,6 +1,5 @@
 <?xml version="1.0"?>
 <robot xmlns:xacro="http://ros.org/wiki/xacro">
-  <xacro:include filename="$(find abb_resources)/urdf/common_materials.xacro"/>
-  <xacro:include filename="$(find pick_and_place_env)/urdf/colours/colours.xacro"/>
+  <xacro:include filename="$(find pick_and_place_env)/urdf/colours/specific_colours.xacro"/>
   <xacro:macro name="abb_irb1200_5_90">
     <!--  -->
@@ -8,18 +7,4 @@
     <!--  -->
     <!-- Robotic arm link list -->
-    <!-- BASE -->
-    <link name="base">
-      <visual name="visual">
-        <geometry>
-          <mesh filename="package://abb_irb1200_support/meshes/irb1200_5_90/visual/robot_stand.stl" scale = "0.001 0.001 0.001"/>
-        </geometry>
-        <xacro:colour_gray_50p/>
-      </visual>
-      <collision name="collision">
-        <geometry>
-          <mesh filename="package://abb_irb1200_support/meshes/irb1200_5_90/visual/robot_stand.stl" scale = "0.001 0.001 0.001"/>
-        </geometry>
-      </collision>
-    </link>
     <!-- BASE_LINK -->
     <link name="base_link">
@@ -33,4 +18,5 @@
           <mesh filename="package://abb_irb1200_support/meshes/irb1200_5_90/collision/base_link.stl"/>
         </geometry>
+        <xacro:collision_colour />
       </collision>
       <inertial>
@@ -46,4 +32,5 @@
           <mesh filename="package://abb_irb1200_support/meshes/irb1200_5_90/visual/link_1.dae"/>
         </geometry>
+        <xacro:collision_colour />
       </visual>
       <collision>
@@ -64,4 +51,5 @@
           <mesh filename="package://abb_irb1200_support/meshes/irb1200_5_90/visual/link_2.dae"/>
         </geometry>
+        <xacro:collision_colour />
       </visual>
       <collision name="collision">
@@ -82,5 +70,5 @@
           <mesh filename="package://abb_irb1200_support/meshes/irb1200_5_90/visual/link_3.dae"/>
         </geometry>
-        <xacro:colour_orange />
+        <xacro:collision_colour />
       </visual>
       <collision name="collision">
@@ -101,4 +89,5 @@
           <mesh filename="package://abb_irb1200_support/meshes/irb1200_5_90/visual/link_4.dae"/>
         </geometry>
+        <xacro:collision_colour />
       </visual>
       <collision name="collision">
@@ -119,4 +108,5 @@
           <mesh filename="package://abb_irb1200_support/meshes/irb1200_5_90/visual/link_5.dae"/>
         </geometry>
+        <xacro:collision_colour />
       </visual>
       <collision name="collision">
@@ -137,4 +127,5 @@
           <mesh filename="package://abb_irb1200_support/meshes/irb1200_5_90/visual/link_6.dae"/>
         </geometry>
+        <xacro:collision_colour />
       </visual>
       <collision name="collision">
@@ -149,4 +140,5 @@
       </inertial>
     </link>
+    <link name="tool0" />
     <!-- End of robotic arm link list -->
     <!--  -->
@@ -158,8 +150,8 @@
     <!--  -->
     <!-- JOINT BASE_LINK -->
-    <joint type="fixed" name="base_link">
-      <origin xyz="0.275 0.275 0.726" rpy="0 0 0"/>
+    <joint name="Room_to_base_link" type="fixed" >
+      <origin xyz="0 0 0.726" rpy="0 0 0"/>
       <axis xyz="0 0 0"/>
-      <parent link="base"/>
+      <parent link="RoomComponents"/>
       <child link="base_link"/>
     </joint>
@@ -219,4 +211,10 @@
     </joint>
     <!-- End of robotic arm joint list -->
+    <!-- ROS-Industrial 'tool0' frame: all-zeros tool frame -->
+    <joint name="link_6-tool0" type="fixed">
+      <origin xyz="0 0 0" rpy="0 ${radians(90)} 0" />
+      <parent link="link_6" />
+      <child link="tool0" />
+    </joint>
   </xacro:macro>
 </robot>

File: src/phoxi_camera/urdf/PhoXi3Dscanner_macro.xacro (robot description, xacro)
@@ -1,46 +1,21 @@
 <?xml version="1.0" ?>
 <robot xmlns:xacro="http://ros.org/wiki/xacro">
-  <xacro:include filename="$(find pick_and_place_env)/urdf/colours/colours.xacro"/>
+  <!-- REMOVE THE LINE BELOW: -->
+  <xacro:include filename="$(find pick_and_place_env)/urdf/colours/specific_colours.xacro"/>
   <xacro:macro name = "PhoXi3Dscanner">
     <!-- link list -->
-    <link name="camera_stand">
+    <link name="PhoXi3Dscanner">
       <visual>
+        <!-- <origin xyz="0 0 0" rpy="0 1.5707 0" /> -->
         <geometry>
-          <mesh filename="package://abb_irb1200_support/meshes/irb1200_5_90/visual/camera_stand.stl" scale = "0.001 0.001 0.001"/>
+          <mesh filename="package://phoxi_camera/meshes/visual/PhoXi3DScannerS.dae" scale = "0.01 0.01 0.01"/>
         </geometry>
-        <!-- <xacro:colour_gray_70p/> -->
       </visual>
       <collision>
+        <!-- <origin xyz="0 0 0" rpy="0 1.5707 0" /> -->
         <geometry>
-          <mesh filename="package://abb_irb1200_support/meshes/irb1200_5_90/visual/camera_stand.stl" scale = "0.001 0.001 0.001"/>
+          <mesh filename="package://phoxi_camera/meshes/collision/PhoXi3DScannerSCollision.stl" scale = "0.001 0.001 0.001"/>
         </geometry>
-      </collision>
-    </link>
-    <link name="camera_support">
-      <visual>
-        <geometry>
-          <mesh filename="package://abb_irb1200_support/meshes/irb1200_5_90/visual/camera_support.stl" scale = "0.001 0.001 0.001"/>
-        </geometry>
-        <!-- <xacro:colour_gray_50p/> -->
-      </visual>
-      <collision>
-        <geometry>
-          <mesh filename="package://abb_irb1200_support/meshes/irb1200_5_90/visual/camera_support.stl" scale = "0.001 0.001 0.001"/>
-        </geometry>
-      </collision>
-    </link>
-    <link name="PhoXi3Dscanner">
-      <visual>
-        <origin xyz="0 0 0" rpy="0 1.5707 0" />
-        <geometry>
-          <mesh filename="package://phoxi_camera/meshes/visual/PhoXi_S.f.STL" scale = "0.001 0.001 0.001"/>
-        </geometry>
-        <xacro:colour_gray_30p/>
-      </visual>
-      <collision>
-        <origin xyz="0 0 0" rpy="0 1.5707 0" />
-        <geometry>
-          <mesh filename="package://phoxi_camera/meshes/collision/PhoXi_L.c.STL" scale = "0.001 0.001 0.001"/>
-        </geometry>
+        <xacro:collision_colour />
       </collision>
     </link>
@@ -50,20 +25,7 @@
     <!--  -->
     <!-- joint list -->
-    <joint name="base_to_camera_stand_joint" type="fixed">
-      <origin xyz="1.535 1.02 0" rpy="0 0 ${pi}"/>
-      <axis xyz="0 0 1"/>
-      <parent link="base"/>
-      <child link="camera_stand"/>
-    </joint>
-    <joint name="camera_stand_to_camera_support_joint" type="fixed">
-      <origin xyz="0.515 0.145 1.202" rpy="0 0 ${pi}"/>
-      <axis xyz="0 0 1"/>
-      <parent link="camera_stand"/>
-      <child link="camera_support"/>
-    </joint>
     <joint name="camera_support_to_PhoXi3Dscanner_joint" type="fixed">
-      <origin xyz="0 0.04 0.02" rpy="${pi} 0 ${-pi/2}"/>
-      <axis xyz="0 0 1"/>
-      <parent link="camera_support"/>
+      <origin xyz="0.6096 -0.49705 1.2235" rpy="${pi/2} 0 ${-pi/2}"/>
+      <parent link="ConveyorAndSupportComponents"/>
       <child link="PhoXi3Dscanner"/>
     </joint>

File: src/pick_and_place_env/urdf/environment.xacro (robot description, xacro)
@@ -1,11 +1,13 @@
 <?xml version="1.0"?>
 <robot name="abb_irb1200_5_90" xmlns:xacro="http://ros.org/wiki/xacro">
+  <xacro:include filename="$(find pick_and_place_env)/urdf/Fixed_parts_macro.xacro"/>
+  <xacro:Fixed_parts/>
   <xacro:include filename="$(find abb_irb1200_support)/urdf/irb1200_5_90_macro.xacro"/>
   <xacro:abb_irb1200_5_90 />
   <xacro:include filename="$(find pick_and_place_env)/urdf/two_finger_gripper_macro.xacro"/>
   <xacro:two_finger_gripper />
+  <!-- <xacro:include filename="$(find pick_and_place_env)/urdf/calibration_tool_macro.xacro"/>
+  <xacro:calibration_tool /> -->
   <xacro:include filename="$(find phoxi_camera)/urdf/PhoXi3Dscanner_macro.xacro"/>
   <xacro:PhoXi3Dscanner />
-  <xacro:include filename="$(find pick_and_place_env)/urdf/conveyor_belt_macro.xacro"/>
-  <xacro:Conveyor_belt/>
 </robot>

File: src/pick_and_place_env/urdf/two_finger_gripper_macro.xacro (robot description, xacro)
@@ -3,4 +3,5 @@
   <xacro:include filename="$(find abb_resources)/urdf/common_materials.xacro"/>
   <xacro:include filename="$(find pick_and_place_env)/urdf/colours/colours.xacro"/>
+  <xacro:include filename="$(find pick_and_place_env)/urdf/colours/specific_colours.xacro"/>
   <xacro:macro name="two_finger_gripper">
     <!--  -->
@@ -11,12 +12,12 @@
       <visual name="visual">
         <geometry>
-          <mesh filename="package://pick_and_place_env/meshes/Common_Flange.stl" scale = "0.001 0.001 0.001"/>
+          <mesh filename="package://pick_and_place_env/meshes/New_meshes/Flange_01.dae" scale = "0.01 0.01 0.01"/>
         </geometry>
-        <!-- <xacro:colour_orange /> -->
       </visual>
       <collision name="collision">
         <geometry>
-          <mesh filename="package://pick_and_place_env/meshes/Common_Flange.stl" scale = "0.001 0.001 0.001"/>
+          <mesh filename="package://pick_and_place_env/meshes/updated_meshes/Flange_01Collision.stl" scale = "0.001 0.001 0.001"/>
         </geometry>
+        <xacro:collision_colour />
       </collision>
       <inertial>
@@ -28,12 +29,12 @@
       <visual name="visual">
         <geometry>
-          <mesh filename="package://pick_and_place_env/meshes/PB-0013_Flange.stl" scale = "0.001 0.001 0.001"/>
+          <mesh filename="package://pick_and_place_env/meshes/New_meshes/Flange_02.dae" scale = "0.01 0.01 0.01"/>
         </geometry>
-        <!-- <xacro:colour_white /> -->
       </visual>
       <collision name="collision">
         <geometry>
-          <mesh filename="package://pick_and_place_env/meshes/PB-0013_Flange.stl" scale = "0.001 0.001 0.001"/>
+          <mesh filename="package://pick_and_place_env/meshes/updated_meshes/Flange_02Collision.stl" scale = "0.001 0.001 0.001"/>
         </geometry>
+        <xacro:collision_colour />
       </collision>
       <inertial>
@@ -47,10 +48,11 @@
           <mesh filename="package://pick_and_place_env/meshes/PB-0013_Base.stl" scale = "0.001 0.001 0.001"/>
         </geometry>
-        <!-- <xacro:colour_gray_20p /> -->
+        <xacro:colour_gray_20p />
       </visual>
       <collision name="collision">
         <geometry>
-          <mesh filename="package://pick_and_place_env/meshes/PB-0013_Base.stl" scale = "0.001 0.001 0.001"/>
+          <mesh filename="package://pick_and_place_env/meshes/updated_meshes/PB-0013BaseCollision.stl" scale = "0.001 0.001 0.001"/>
         </geometry>
+        <xacro:collision_colour />
       </collision>
       <inertial>
@@ -64,10 +66,11 @@
           <mesh filename="package://pick_and_place_env/meshes/PB-0013_Left.stl" scale = "0.001 0.001 0.001"/>
         </geometry>
-        <!-- <xacro:colour_gray_40p /> -->
+        <xacro:colour_gray_40p />
       </visual>
       <collision name="collision">
         <geometry>
-          <mesh filename="package://pick_and_place_env/meshes/PB-0013_Left.stl" scale = "0.001 0.001 0.001"/>
+          <mesh filename="package://pick_and_place_env/meshes/updated_meshes/PB-0013LeftCollision.stl" scale = "0.001 0.001 0.001"/>
         </geometry>
+        <xacro:collision_colour />
       </collision>
       <inertial>
@@ -81,10 +84,11 @@
           <mesh filename="package://pick_and_place_env/meshes/PB-0013_Right.stl" scale = "0.001 0.001 0.001"/>
         </geometry>
-        <!-- <xacro:colour_gray_40p /> -->
+        <xacro:colour_gray_40p />
       </visual>
       <collision name="collision">
         <geometry>
-          <mesh filename="package://pick_and_place_env/meshes/PB-0013_Right.stl" scale = "0.001 0.001 0.001"/>
+          <mesh filename="package://pick_and_place_env/meshes/updated_meshes/PB-0013RightCollision.stl" scale = "0.001 0.001 0.001"/>
         </geometry>
+        <xacro:collision_colour />
       </collision>
       <inertial>
@@ -99,6 +103,6 @@
     <!-- Gripper joint list -->
     <joint type="fixed" name="joint_flange_1">
-      <origin xyz="0 -0.02 0.02" rpy="0 ${pi/2} 0"/>
-      <parent link="link_6"/>
+      <origin xyz="0 0 0" rpy="0 0 0"/>
+      <parent link="tool0"/>
       <child link="link_flange_1"/>
     </joint>
@@ -109,5 +113,5 @@
     </joint>
     <joint type="fixed" name="joint_tool_base">
-      <origin xyz="0.02 0.02 0.151" rpy="${pi} 0 0"/>
+      <origin xyz="0 0 0.116" rpy="${pi} 0 ${pi/2}"/>
       <parent link="link_flange_2"/>
       <child link="link_tool_base"/>
