Commit message: Working

File: src/abb_robot_arm/abb_irb1200_support/urdf/irb1200_5_90_macro.xacro (robot description, xacro)
@@ -150,15 +150,8 @@
     <!--  -->
     <!-- JOINT BASE_LINK -->
-<<<<<<< HEAD
     <joint name="Room_to_base_link" type="fixed" >
       <origin xyz="0 0 0.726" rpy="0 0 0"/>
       <axis xyz="0 0 0"/>
       <parent link="RoomComponents"/>
-=======
-    <joint type="fixed" name="base_link">
-      <origin xyz="0 0 0.726" rpy="0 0 0"/>
-      <axis xyz="0 0 0"/>
-      <parent link="Fixed_frame"/>
->>>>>>> 111af121142ca18e335d97f9c4da8065ef0ffcb4
       <child link="base_link"/>
     </joint>

File: src/phoxi_camera/urdf/PhoXi3Dscanner_macro.xacro (robot description, xacro)
@@ -15,9 +15,5 @@
         <!-- <origin xyz="0 0 0" rpy="0 1.5707 0" /> -->
         <geometry>
-<<<<<<< HEAD
           <mesh filename="package://phoxi_camera/meshes/collision/PhoXi3DScannerSCollision.stl" scale = "0.001 0.001 0.001"/>
-=======
-          <mesh filename="package://phoxi_camera/meshes/collision/PhoXi_S.c.STL" scale = "0.001 0.001 0.001"/>
->>>>>>> 111af121142ca18e335d97f9c4da8065ef0ffcb4
         </geometry>
         <xacro:collision_colour />
@@ -29,13 +25,7 @@
     <!--  -->
     <!-- joint list -->
-<<<<<<< HEAD
     <joint name="camera_support_to_PhoXi3Dscanner_joint" type="fixed">
       <origin xyz="0.6096 -0.49705 1.2235" rpy="${pi/2} 0 ${-pi/2}"/>
       <parent link="ConveyorAndSupportComponents"/>
-=======
-    <joint name="camera_support_to_PhoXi3Dscanner_joint" type="fixed">
-      <origin xyz="0.745 0.640 1.231" rpy="${pi} 0 ${-pi/2}"/>
-      <parent link="Fixed_frame"/>
->>>>>>> 111af121142ca18e335d97f9c4da8065ef0ffcb4
       <child link="PhoXi3Dscanner"/>
     </joint>

File: src/pick_and_place_env/urdf/Fixed_parts_macro.xacro (robot description, xacro)
@@ -1,5 +1,4 @@
 <?xml version="1.0" ?>
 <robot xmlns:xacro="http://ros.org/wiki/xacro">
-<<<<<<< HEAD
   <xacro:include filename="$(find pick_and_place_env)/urdf/colours/specific_colours.xacro"/>
   <xacro:macro name = "Fixed_parts">
@@ -9,18 +8,8 @@
         <geometry>
           <mesh filename="package://pick_and_place_env/meshes/updated_meshes/RoomComponents.dae" scale = "0.01 0.01 0.01"/>
-=======
-  <xacro:include filename="$(find pick_and_place_env)/urdf/colours/colours.xacro"/>
-  <xacro:macro name = "Fixed_parts">
-    <!-- link list -->
-    <link name="Fixed_frame">
-      <visual>
-        <geometry>
-          <mesh filename="package://pick_and_place_env/meshes/New_meshes/Fixed_parts_pillot_line.dae" scale = "0.01 0.01 0.01"/>
->>>>>>> 111af121142ca18e335d97f9c4da8065ef0ffcb4
         </geometry>
       </visual>
       <collision name="collision">
         <geometry>
-<<<<<<< HEAD
           <mesh filename="package://pick_and_place_env/meshes/updated_meshes/RoomCollision.stl" scale = "0.001 0.001 0.001"/>
         </geometry>
@@ -71,11 +60,4 @@
     </joint>
     <!-- end of joint list -->
-=======
-          <mesh filename="package://pick_and_place_env/meshes/New_meshes/Fixed_parts_pillot_line.dae" scale = "0.01 0.01 0.01"/>
-        </geometry>
-      </collision>
-    </link>
-    <!-- end of link list -->
->>>>>>> 111af121142ca18e335d97f9c4da8065ef0ffcb4
   </xacro:macro>
 </robot>

File: src/pick_and_place_env/urdf/two_finger_gripper_macro.xacro (robot description, xacro)
@@ -14,8 +14,4 @@
           <mesh filename="package://pick_and_place_env/meshes/New_meshes/Flange_01.dae" scale = "0.01 0.01 0.01"/>
         </geometry>
-<<<<<<< HEAD
-=======
-        <xacro:colour_orange />
->>>>>>> 111af121142ca18e335d97f9c4da8065ef0ffcb4
       </visual>
       <collision name="collision">
@@ -35,8 +31,4 @@
           <mesh filename="package://pick_and_place_env/meshes/New_meshes/Flange_02.dae" scale = "0.01 0.01 0.01"/>
         </geometry>
-<<<<<<< HEAD
-=======
-        <xacro:colour_white />
->>>>>>> 111af121142ca18e335d97f9c4da8065ef0ffcb4
       </visual>
       <collision name="collision">
