Commit message: Updating

File: src/phoxi_camera/urdf/PhoXi3Dscanner_macro.xacro (robot description, xacro)
@@ -26,5 +26,5 @@
     <!-- joint list -->
     <joint name="camera_support_to_PhoXi3Dscanner_joint" type="fixed">
-      <origin xyz="0.6096 -0.49705 1.2235" rpy="${pi/2} 0 ${-pi/2}"/>
+      <origin xyz="0.6096 -0.49705 1.2235" rpy="${pi} 0 ${-pi}"/>
       <parent link="ConveyorAndSupportComponents"/>
       <child link="PhoXi3Dscanner"/>
